Commit message: change folder

File: ur_description/urdf/ur_macro.xacro (robot description, xacro)
@@ -70,6 +70,7 @@
         <origin xyz="0 0 0" rpy="0 0 ${pi}"/>
         <geometry>
-          <xacro:get_mesh name="base" type="visual"/>
-        </geometry>
+					<mesh
+						filename="package://ur_description/meshes/ur5e/visual/base.dae" />
+				</geometry>
       </visual>
       <collision>
@@ -87,5 +88,6 @@
         <origin xyz="0 0 0" rpy="0 0 ${pi}"/>
         <geometry>
-          <xacro:get_mesh name="shoulder" type="visual"/>
+          <mesh
+            filename="package://ur_description/meshes/ur5e/visual/shoulder.dae" />
         </geometry>
       </visual>
@@ -104,5 +106,6 @@
         <origin xyz="0 0 ${shoulder_offset}" rpy="${pi/2} 0 ${-pi/2}"/>
         <geometry>
-          <xacro:get_mesh name="upper_arm" type="visual"/>
+          <mesh
+            filename="package://ur_description/meshes/ur5e/visual/upperarm.dae" />
         </geometry>
       </visual>
@@ -121,5 +124,6 @@
         <origin xyz="0 0 ${elbow_offset}" rpy="${pi/2} 0 ${-pi/2}"/>
         <geometry>
-          <xacro:get_mesh name="forearm" type="visual"/>
+          <mesh
+            filename="package://ur_description/meshes/ur5e/visual/forearm.dae" />
         </geometry>
       </visual>
@@ -139,5 +143,6 @@
       	<origin xyz="0 0 ${visual_params}" rpy="${pi/2} 0 0"/>
         <geometry>
-          <xacro:get_mesh name="wrist_1" type="visual"/>
+          <mesh
+            filename="package://ur_description/meshes/ur5e/visual/wrist1.dae" />
         </geometry>
       </visual>
@@ -157,5 +162,6 @@
         <origin xyz="0 0 ${visual_params}" rpy="0 0 0"/>
         <geometry>
-          <xacro:get_mesh name="wrist_2" type="visual"/>
+          <mesh
+            filename="package://ur_description/meshes/ur5e/visual/wrist2.dae" />
         </geometry>
       </visual>
@@ -175,5 +181,6 @@
         <origin xyz="0 0 ${visual_params}" rpy="${pi/2} 0 0"/>
         <geometry>
-          <xacro:get_mesh name="wrist_3" type="visual"/>
+          <mesh
+            filename="package://meshes/ur5e/visual/wrist3.dae" />
         </geometry>
       </visual>
